File: ROV - Light Module/KiCAD/Arduino Driver PCB.kicad_sch (KiCad schematic)
At the start: 24 parts, among them J1 AVR UPDI Header, J4 Bottom - Middle, J6 Main In, U2 ATtiny1614-Arduino, U3 AP63205WU, U6 MAX3072E

Commit message: design review
Other:
- note added: "V_in 12-18 V nominal, 24 VDC Max"
Changed lines of the file:
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@@
 	(generator_version "10.0")
 	(paper "A4")
+	(text "V_in 12-18 V nominal, 24 VDC Max"
+		(exclude_from_sim no)
+		(at 44.196 59.436 0)
+		(effects
+			(font
+				(size 1.524 1.524)
+			)
+		)
+	)
 	(text "The Feedback LED is not part of the AVR HDPI header standard, however, I\nhave included it on the un-used pin so that I can have a status/feedback\nLED for visual feedback from the microcontroller."
 		(exclude_from_sim no)
@@
 		(length 1)
 		(shape round)
+		(at 43.18 34.29 0)
+		(fields_autoplaced yes)
+		(effects
+			(font
+				(size 1.524 1.524)
+				(color 255 153 0 1)
+			)
+			(justify left bottom)
+		)
+		(property "Netclass" "1 oz - 1 A"
+			(at 43.8099 33.29 0)
+			(show_name no)
+			(do_not_autoplace no)
+			(effects
+				(font
+					(size 0.5 0.5)
+				)
+				(justify left bottom)
+			)
+		)
+		(property "Component Class" ""
+			(at -201.93 6.35 0)
+			(show_name no)
+			(do_not_autoplace no)
+			(effects
+				(font
+					(size 1.27 1.27)
+					(italic yes)
+				)
+			)
+		)
+	)
+	(netclass_flag ""
+		(length 1)
+		(shape round)
 		(at 106.68 93.98 0)
 		(fields_autoplaced yes)
@@
 		(length 1)
 		(shape round)
-		(at 43.18 34.29 0)
-		(fields_autoplaced yes)
-		(effects
-			(font
-				(size 1.524 1.524)
-				(color 255 153 0 1)
-			)
-			(justify left bottom)
-		)
-		(property "Netclass" "1 oz - 2 A"
-			(at 43.8099 33.29 0)
-			(show_name no)
-			(do_not_autoplace no)
-			(effects
-				(font
-					(size 0.5 0.5)
-				)
-				(justify left bottom)
-			)
-		)
-		(property "Component Class" ""
-			(at -201.93 6.35 0)
-			(show_name no)
-			(do_not_autoplace no)
-			(effects
-				(font
-					(size 1.27 1.27)
-					(italic yes)
-				)
-			)
-		)
-	)
-	(netclass_flag ""
-		(length 1)
-		(shape round)
-		(at 153.67 31.75 0)
-		(fields_autoplaced yes)
-		(effects
-			(font
-				(size 1.524 1.524)
-				(color 255 153 0 1)
-			)
-			(justify left bottom)
-		)
-		(property "Netclass" "1 oz - 2 A"
-			(at 154.2999 30.75 0)
-			(show_name no)
-			(do_not_autoplace no)
-			(effects
-				(font
-					(size 0.5 0.5)
-				)
-				(justify left bottom)
-			)
-		)
-		(property "Component Class" ""
-			(at -91.44 3.81 0)
-			(show_name no)
-			(do_not_autoplace no)
-			(effects
-				(font
-					(size 1.27 1.27)
-					(italic yes)
-				)
-			)
-		)
-	)
-	(netclass_flag ""
-		(length 1)
-		(shape round)
 		(at 251.46 154.94 0)
 		(fields_autoplaced yes)
@@
 		(length 1)
 		(shape round)
+		(at 146.05 31.75 0)
+		(fields_autoplaced yes)
+		(effects
+			(font
+				(size 1.524 1.524)
+				(color 255 153 0 1)
+			)
+			(justify left bottom)
+		)
+		(property "Netclass" "1 oz - 1 A"
+			(at 146.6799 30.75 0)
+			(show_name no)
+			(do_not_autoplace no)
+			(effects
+				(font
+					(size 0.5 0.5)
+				)
+				(justify left bottom)
+			)
+		)
+		(property "Component Class" ""
+			(at -99.06 3.81 0)
+			(show_name no)
+			(do_not_autoplace no)
+			(effects
+				(font
+					(size 1.27 1.27)
+					(italic yes)
+				)
+			)
+		)
+	)
+	(netclass_flag ""
+		(length 1)
+		(shape round)
 		(at 106.68 91.44 0)
 		(fields_autoplaced yes)
@@
 		(length 1)
 		(shape round)
-		(at 50.8 34.29 0)
-		(fields_autoplaced yes)
-		(effects
-			(font
-				(size 1.524 1.524)
-				(color 255 153 0 1)
-			)
-			(justify left bottom)
-		)
-		(property "Netclass" "1 oz - 2 A"
-			(at 51.4299 33.29 0)
-			(show_name no)
-			(do_not_autoplace no)
-			(effects
-				(font
-					(size 0.5 0.5)
-				)
-				(justify left bottom)
-			)
-		)
-		(property "Component Class" ""
-			(at -194.31 6.35 0)
-			(show_name no)
-			(do_not_autoplace no)
-			(effects
-				(font
-					(size 1.27 1.27)
-					(italic yes)
-				)
-			)
-		)
-	)
-	(netclass_flag ""
-		(length 1)
-		(shape round)
 		(at 64.77 104.14 0)
 		(fields_autoplaced yes)
@@
 		(length 1)
 		(shape round)
+		(at 165.1 31.75 0)
+		(fields_autoplaced yes)
+		(effects
+			(font
+				(size 1.524 1.524)
+				(color 255 153 0 1)
+			)
+			(justify left bottom)
+		)
+		(property "Netclass" "1 oz - 1 A"
+			(at 165.7299 30.75 0)
+			(show_name no)
+			(do_not_autoplace no)
+			(effects
+				(font
+					(size 0.5 0.5)
+				)
+				(justify left bottom)
+			)
+		)
+		(property "Component Class" ""
+			(at -80.01 3.81 0)
+			(show_name no)
+			(do_not_autoplace no)
+			(effects
+				(font
+					(size 1.27 1.27)
+					(italic yes)
+				)
+			)
+		)
+	)
+	(netclass_flag ""
+		(length 1)
+		(shape round)
 		(at 146.05 34.29 0)
 		(fields_autoplaced yes)
@@
 		(length 1)
 		(shape round)
-		(at 205.74 31.75 0)
-		(fields_autoplaced yes)
-		(effects
-			(font
-				(size 1.524 1.524)
-				(color 255 153 0 1)
-			)
-			(justify left bottom)
-		)
-		(property "Netclass" "1 oz - 2 A"
-			(at 206.3699 30.75 0)
-			(show_name no)
-			(do_not_autoplace no)
-			(effects
-				(font
-					(size 0.5 0.5)
-				)
-				(justify left bottom)
-			)
-		)
-		(property "Component Class" ""
-			(at -39.37 3.81 0)
-			(show_name no)
-			(do_not_autoplace no)
+		(at 50.8 34.29 0)
+		(fields_autoplaced yes)
+		(effects
+			(font
+				(size 1.524 1.524)
+				(color 255 153 0 1)
+			)
+			(justify left bottom)
+		)
+		(property "Netclass" "1 oz - 1 A"
+			(at 51.4299 33.29 0)
+			(show_name no)
+			(do_not_autoplace no)
+			(effects
+				(font
+					(size 0.5 0.5)
+				)
+				(justify left bottom)
+			)
+		)
+		(property "Component Class" ""
+			(at -194.31 6.35 0)
+			(show_name no)
+			(do_not_autoplace no)

Commit message: updates
Parts:
- removed JP1: TX, Jumper:SolderJumper-2_P1.3mm_Open_TrianglePad1.0x1.5mm, symbol Jumper:SolderJumper_2_Open
- removed JP3: RX, Jumper:SolderJumper-2_P1.3mm_Open_TrianglePad1.0x1.5mm, symbol Jumper:SolderJumper_2_Open
- C3: value 100nF -> 10pF
- J1: footprint Connector_PinHeader_2.54mm:PinHeader_2x03_P2.54mm_Vertical -> Connector_PinHeader_1.27mm:PinHeader_2x03_P1.27mm_Vertical_SMD
- J4: value Bottom - Middle -> Conn_02x05_Odd_Even; footprint Connector_PinSocket_1.27mm:PinSocket_2x06_P1.27mm_Vertical_SMD -> Connector_PinSocket_1.27mm:PinSocket_2x05_P1.27mm_Vertical_SMD; symbol Connector_Generic:Conn_02x06_Odd_Even -> Connector_Generic:Conn_02x05_Odd_Even
Connections:
- net +5V: now also J4.3 (Pin_3); no longer J4.5 (Pin_5), J4.7 (Pin_7)
- net A9/D9: now also J4.7 (Pin_7); no longer J4.8 (Pin_8)
- net Data_A: now also J6.4 (Pin_4); no longer J6.3 (Pin_3)
- net Data_B: now also J6.3 (Pin_3); no longer J6.4 (Pin_4)
- net LED_PWM: now also J4.6 (Pin_6); no longer J4.9 (Pin_9)
- net NeoPixle: now also J4.5 (Pin_5); no longer J4.6 (Pin_6)
- net SCL: now also J4.8 (Pin_8); no longer J4.10 (Pin_10)
- net SDA: now also J4.10 (Pin_10); no longer J4.12 (Pin_12)
- net STATUS_LED: now also J4.9 (Pin_9); no longer J4.11 (Pin_11)
- net V_in: no longer J4.3 (Pin_3)
- net V_Supply: now reaches D5.2 (A), J6.1 (Pin_1)
Other:
- note added: "Large copper pour rather than tracks!"
- moved on the sheet: C3, C4, C9, J6, U6

Commit message: cleanup
Parts:
- removed J4: Conn_02x05_Odd_Even, Connector_PinSocket_1.27mm:PinSocket_2x05_P1.27mm_Vertical_SMD, symbol Connector_Generic:Conn_02x05_Odd_Even
- J6: footprint Connector_PinHeader_2.54mm:PinHeader_1x05_P2.54mm_Vertical -> Connector_PinHeader_2.54mm:PinHeader_1x05_P2.54mm_Vertical_SMD_Pin1Left
- R9: value 37k -> 51k
- U6: value MAX3072E -> ADM485
Connections:
- net SERIAL_RX: now also U6.1 (RO); no longer U6.4 (DI)
- net SERIAL_TX: now also U6.4 (DI); no longer U6.1 (RO)
- net STATUS_LED: no longer U2.3 (~A1/D1)
- net LED_PWM renamed ~A0/D0
- net NeoPixle renamed ~A10/D10_SCK
- new net ~A1/D1: U2.3 (~A1/D1)
Other:
- note added: "### V_in Measurement The input voltage is measured through a 51 kΩ / 12 kΩ resistor divider. The expected ADC voltage is: `Vmeasure = V_in × 12 / (51 + 12)` | Input voltage | Expected Vmeasure | |---:|---:| | 12 VDC | 2.29 V | | 18 VDC | 3.43 V | | 24 VDC | 4.57 V | These values assume ideal resistor values. Component tolerance and supply variation will introduce small differences."
