File: ROV - Light Module/KiCAD/Arduino Driver PCB.kicad_sch (KiCad schematic)
At the start: 21 parts, among them J1 AVR UPDI Header, J6 Main In, U2 ATtiny1614-Arduino, U3 AP63205WU, U6 MAX13487E

Commit message: massive cleanup
Other:
- note added: "The Feedback LED (built in) is not part of the AVR UPDI header standard, however, I have included it on the un-used pin so that I can have a status/feedback LED for visual feedback from the microcontroller."
- note removed: "The Feedback LED is not part of the AVR HDPI header standard, however, I have included it on the un-used pin so that I can have a status/feedback LED for visual feedback from the microcontroller."
