File: ROV - Conductivity Temperature and Depth Transducer/KiCAD/ROV CTD.kicad_sch (KiCad schematic)
At the start: 39 parts, among them J2 Temp, J4 Bottom - Middle, J6 Main In, J7 Bottom - Middle, J8 Middle - Top, J9 Top - Middle, U2 ATtiny1614-Arduino, U3 AP63205WU, U5 RT9166/A, U6 MAX3072E

Commit message: update PCBs
Parts:
- removed C10, C9: 47uF, Capacitor_SMD:C_0805_2012Metric_Pad1.18x1.45mm_HandSolder, symbol Device:C_Small
- removed C13, C15, C3, C5: 100nF, Capacitor_SMD:C_0805_2012Metric_Pad1.18x1.45mm_HandSolder, symbol Device:C_Small
- removed C14: 10uF, Capacitor_SMD:C_0805_2012Metric_Pad1.18x1.45mm_HandSolder, symbol Device:C_Small
- removed C16, C17: 22uF, Capacitor_SMD:C_0805_2012Metric_Pad1.18x1.45mm_HandSolder, symbol Device:C_Small
- removed C4, C6: 10pF, Capacitor_SMD:C_0805_2012Metric_Pad1.18x1.45mm_HandSolder, symbol Device:C_Small
- removed D10: 5V, LED_SMD:LED_0805_2012Metric_Pad1.15x1.40mm_HandSolder, symbol Device:LED_Small_Filled
- removed D4: Status, LED_SMD:LED_0805_2012Metric_Pad1.15x1.40mm_HandSolder, symbol Device:LED_Small_Filled
- removed D5: CZRB5370B-HF, Diode_SMD:D_SMB_Handsoldering, symbol Partsbox:CZRB5370B-HF
- removed J6: Main In, Connector_PinHeader_2.54mm:PinHeader_1x05_P2.54mm_Vertical, symbol Connector:Conn_01x05_Pin
- removed J9: Top - Middle, Connector_PinHeader_1.27mm:PinHeader_2x06_P1.27mm_Vertical_SMD, symbol Connector_Generic:Conn_02x06_Odd_Even
- removed JP1: TX, Jumper:SolderJumper-2_P1.3mm_Open_TrianglePad1.0x1.5mm, symbol Jumper:SolderJumper_2_Open
- removed JP2: RX, Jumper:SolderJumper-2_P1.3mm_Open_TrianglePad1.0x1.5mm, symbol Jumper:SolderJumper_2_Open
- removed L2: 4.7uH, Inductor_SMD:L_Vishay_IHLP-1212, symbol Device:L_Small
- removed R10: 12k, Resistor_SMD:R_0805_2012Metric_Pad1.20x1.40mm_HandSolder, symbol Device:R_Small
- removed R11: 1k, Resistor_SMD:R_0805_2012Metric_Pad1.20x1.40mm_HandSolder, symbol Device:R_Small
- removed R7: 520, Resistor_SMD:R_0805_2012Metric_Pad1.20x1.40mm_HandSolder, symbol Device:R_Small
- removed R9: 37k, Resistor_SMD:R_0805_2012Metric_Pad1.20x1.40mm_HandSolder, symbol Device:R_Small
- removed U2: ATtiny1614-Arduino, Package_SO:SOIC-14_3.9x8.7mm_P1.27mm, symbol KiCad Symbols:ATtiny1614-Arduino
- removed U3: AP63205WU, Package_TO_SOT_SMD:TSOT-23-6, symbol Regulator_Switching:AP63200WU
- removed U6: MAX3072E, Package_SO:SOIC-8_3.9x4.9mm_P1.27mm, symbol Interface_UART:MAX3072E
- added J5: Conn_02x05_Odd_Even, Connector_PinSocket_1.27mm:PinSocket_2x05_P1.27mm_Vertical_SMD, symbol Connector_Generic:Conn_02x05_Odd_Even
Connections:
- net +5V: now also J5.3 (Pin_3)
- net GND: now also J5.2 (Pin_2), J5.4 (Pin_4)
- net Top_TDS: now also J5.6 (Pin_6)
- net Top_Temp: now also J5.5 (Pin_5)
- net V_in: now also J5.1 (Pin_1)
- new net SCL: J5.8 (Pin_8)
- new net SDA: J5.10 (Pin_10)
- new net STATUS_LED: J5.9 (Pin_9)
- new net Top_TDS_En: J5.7 (Pin_7)
- no-connect marks 0 -> 1
Other:
- added sheet Arduino Driver PCB (Arduino Driver PCB.kicad_sch)

Commit message: massive cleanup
Parts:
- removed J4: Bottom - Middle, Connector_PinSocket_1.27mm:PinSocket_2x06_P1.27mm_Vertical_SMD, symbol Connector_Generic:Conn_02x06_Odd_Even
- removed J7: Bottom - Middle, Connector_PinHeader_1.27mm:PinHeader_2x06_P1.27mm_Vertical_SMD, symbol Connector_Generic:Conn_02x06_Odd_Even
- removed J8: Middle - Top, Connector_PinSocket_1.27mm:PinSocket_2x06_P1.27mm_Vertical_SMD, symbol Connector_Generic:Conn_02x06_Odd_Even
- added D7: Status_Led, LED_SMD:LED_0805_2012Metric_Pad1.15x1.40mm_HandSolder, symbol Device:LED_Small_Filled
- added J3, J4: Conn_02x05_Odd_Even, Connector_PinHeader_1.27mm:PinHeader_2x05_P1.27mm_Vertical_SMD, symbol Connector_Generic:Conn_02x05_Odd_Even
- added J5: Conn_02x05_Odd_Even, Connector_PinSocket_1.27mm:PinSocket_2x05_P1.27mm_Vertical_SMD, symbol Connector_Generic:Conn_02x05_Odd_Even
- added R21: 1k, Resistor_SMD:R_0805_2012Metric_Pad1.20x1.40mm_HandSolder, symbol Device:R_Small
- renumbered C30 to C1, C31 to C2, C29 to C3, C32 to C4, C21 to C5, J2 to J1, J5 to J2, R25 to R1, U5 to U1
Connections:
- net +5V: no longer C1.1, C2.1, R1.2, U1.3 (IN)
- net Bot_Probe_1: now also H2.1, J4.5 (Pin_5); no longer H1.1
- net Bot_Probe_2: now also H1.1, J4.6 (Pin_6); no longer H2.1
- net Bot_SCL: now also J4.8 (Pin_8)
- net Bot_SDA: now also J4.10 (Pin_10)
- net Bot_Temp: now also J4.7 (Pin_7)
- net GND: now also D7.1 (K), J3.2 (Pin_2), J3.4 (Pin_4), J4.2 (Pin_2), J4.4 (Pin_4), J5.2 (Pin_2), J5.4 (Pin_4)
- net Mid_Probe_1: now also J5.5 (Pin_5)
- net Mid_Probe_2: now also J5.6 (Pin_6)
- net Mid_SCL: now also J3.8 (Pin_8), J5.8 (Pin_8)
- net Mid_SDA: now also J3.10 (Pin_10), J5.10 (Pin_10)
- net Mid_TDS: now also J3.6 (Pin_6)
- net Mid_Temp: now also J3.5 (Pin_5), J5.7 (Pin_7)
- net Top_TDS_En renamed Top_TDS_OSC
- new net: D7.2 (A), R21.2
- new net +5V_Bot: C1.1, C2.1, J4.3 (Pin_3), R1.2, U1.3 (IN)
- new net +5V_Mid: J3.3 (Pin_3), J5.3 (Pin_3)
- new net Bot_Status_LED: J4.9 (Pin_9), R21.1
- new net Mid_Status_LED: J3.9 (Pin_9), J5.9 (Pin_9)
- new net Mid_TDS_OSC: J3.7 (Pin_7)
- no-connect marks 1 -> 4
Other:
- moved on the sheet: H1, H2
