File: ROV - Conductivity Temperature and Depth Transducer/KiCAD/Arduino Driver PCB.kicad_sch (KiCad schematic)
At the start: 21 parts, among them J1 AVR UPDI Header, J6 Main In, U2 ATtiny1614-Arduino, U3 AP63205WU, U6 MAX13487E

Commit message: massive cleanup
Parts:
- renumbered C4 to C20, C13 to C21, C14 to C22, C15 to C23, C16 to C24, C17 to C25, C9 to C26, C3 to C27, D5 to D4, D4 to D5, D10 to D6, J1 to J7, L2 to L1, R9 to R17, R10 to R18, R7 to R19, R11 to R20, U2 to U4, U3 to U5
Other:
- note added: "The Feedback LED is not part of the AVR UPDI header standard, however, I have included it on the un-used pin so that I can have a status/feedback LED for visual feedback from the microcontroller."
- note removed: "The Feedback LED is not part of the AVR HDPI header standard, however, I have included it on the un-used pin so that I can have a status/feedback LED for visual feedback from the microcontroller."

Commit message: working on CDT
Parts:
- renumbered C21 to C13, C22 to C14, C23 to C15, C24 to C16, C25 to C17, C27 to C3, C20 to C4, C26 to C9, D6 to D10, D5 to D4, D4 to D5, J7 to J1, L1 to L2, R18 to R10, R20 to R11, R19 to R7, R17 to R9, U4 to U2, U5 to U3
Other:
- note added: "The Feedback LED (built in) is not part of the AVR UPDI header standard, however, I have included it on the un-used pin so that I can have a status/feedback LED for visual feedback from the microcontroller."
- note removed: "The Feedback LED is not part of the AVR UPDI header standard, however, I have included it on the un-used pin so that I can have a status/feedback LED for visual feedback from the microcontroller."
