File: ROV - Conductivity Temperature and Depth Transducer/KiCAD/Conductivity Transducer.kicad_sch (KiCad schematic)
At the start: 28 parts, among them U1 LMV324, U4 LM2664

Commit message: massive cleanup
Parts:
- renumbered C11 to C10, C27 to C11, C20 to C13, C28 to C14, C23 to C15, C24 to C16, C25 to C17, C26 to C18, C22 to C19, C18 to C8, C19 to C9, D9 to D3, R20 to R10, R21 to R11, R22 to R12, R23 to R13, R27 to R14, R28 to R15, R24 to R16, R18 to R6, R17 to R7, R26 to R8, R19 to R9, U4 to U2, U1 to U3
Connections:
- net +5V renamed +5V_Mid
Other:
- note added: "Probe is based on the work of Marco Carminati and Paolo Luzzatto-Fegiz, published as Conduino (https://github.com/feslab/conduino), licensed CC BY-SA 4.0 (https://creativecommons.org/licenses/by-sa/4.0/). As modified by the OpenCPD team in Conduino-V01.pdf, also identified as CC BY-SA 4.0. PCB design development based on the DFRobot Gravity EC Sensor DFR0300"
- note removed: "Probe is baised on work done by the Marco Carminati and Paolo Luzzatto-Fegiz. Conduino CC-BY-SA 4.0 (https://github.com/feslab/conduino). As modified by the OpenCPD team CC-BY-SA 4.0 (Conduino-V01.pdf). PCB design development baised on the DFRobot Gravity EC Sensor DFR0300"

Commit message: working on CDT
Parts:
- removed C17: 4.7uF, Capacitor_SMD:C_0805_2012Metric_Pad1.18x1.45mm_HandSolder, symbol Device:C_Small
- removed C18: 100nF, Capacitor_SMD:C_0805_2012Metric_Pad1.18x1.45mm_HandSolder, symbol Device:C_Small
- added C30: 100nF, Capacitor_SMD:C_0805_2012Metric_Pad1.18x1.45mm_HandSolder, symbol Device:C_Small
- renumbered C8 to C21, C9 to C22, C10 to C23, C11 to C24, C12 to C25, C13 to C26, C14 to C27, C15 to C28, C16 to C29, C19 to C32, D2 to D13, D3 to D14, D1 to D2, R7 to R19, R8 to R20, R9 to R22, R10 to R23, R11 to R24, R12 to R25, R13 to R26, R14 to R27, R15 to R28, R16 to R29, U2 to U5, U3 to U7
Connections:
- net +5V_Mid: now also C30.1
- net GND: now also C30.2
