File: ROV - Conductivity Temperature and Depth Transducer/KiCAD/Pressure Transducer.kicad_sch (KiCad schematic)
At the start: 9 parts, among them M2 MS5803-14BA

Commit message: massive cleanup
Parts:
- renumbered C7 to C6, C8 to C7, JP3 to JP1, JP4 to JP2, M2 to M1, R15 to R2, R14 to R3, R12 to R4, R13 to R5
Other:
- note added: "This is based on the SparkFun reference design MS5803-14BA Breakout PCB v10.pdf, licensed CC BY-SA 4.0 (https://creativecommons.org/licenses/by-sa/4.0/)"
- note removed: "This is baised on the reference from SparkFun CC-BY-SA 4.0 (MS5803-14BA Breakout PCB v10.pdf)"
Changed lines of the file:
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@@
 		(company "Philip McGaw")
 	)
-	(text "This is baised on the reference from SparkFun CC-BY-SA 4.0\n(MS5803-14BA Breakout PCB v10.pdf)"
+	(text "This is based on the SparkFun reference design MS5803-14BA Breakout PCB v10.pdf, licensed CC BY-SA 4.0 (https://creativecommons.org/licenses/by-sa/4.0/)"
 		(exclude_from_sim no)
 		(at 184.912 173.99 0)
@@
 		(dnp no)
 		(fields_autoplaced yes)
-		(property "Reference" "R15"
+		(property "Reference" "R2"
 			(at 168.91 72.3899 0)
 			(show_name no)
@@
 			(project "ROV CTD"
 				(path "/4b85b8a1-3b52-4af9-b3a4-471ab529b035/150d263f-d8d0-41bc-b04b-394586738282"
-					(reference "R15")
+					(reference "R2")
 					(unit 1)
 				)
@@
 		(dnp no)
 		(fields_autoplaced yes)
-		(property "Reference" "#PWR026"
+		(property "Reference" "#PWR022"
 			(at 67.31 95.25 0)
 			(hide yes)
@@
 			(project "ROV CTD"
 				(path "/4b85b8a1-3b52-4af9-b3a4-471ab529b035/150d263f-d8d0-41bc-b04b-394586738282"
-					(reference "#PWR026")
+					(reference "#PWR022")
 					(unit 1)
 				)
@@
 		(dnp no)
 		(fields_autoplaced yes)
-		(property "Reference" "R13"
+		(property "Reference" "R5"
 			(at 217.17 72.3899 0)
 			(show_name no)
@@
 			(project "ROV CTD"
 				(path "/4b85b8a1-3b52-4af9-b3a4-471ab529b035/150d263f-d8d0-41bc-b04b-394586738282"
-					(reference "R13")
+					(reference "R5")
 					(unit 1)
 				)
@@
 		(dnp no)
 		(fields_autoplaced yes)
-		(property "Reference" "M2"
+		(property "Reference" "M1"
 			(at 192.4686 71.12 0)
 			(show_name no)
@@
 			(project "ROV CTD"
 				(path "/4b85b8a1-3b52-4af9-b3a4-471ab529b035/150d263f-d8d0-41bc-b04b-394586738282"
-					(reference "M2")
+					(reference "M1")
 					(unit 1)
 				)
@@
 		(dnp no)
 		(fields_autoplaced yes)
-		(property "Reference" "R12"
+		(property "Reference" "R4"
 			(at 208.28 72.3899 0)
 			(show_name no)
@@
 			(project "ROV CTD"
 				(path "/4b85b8a1-3b52-4af9-b3a4-471ab529b035/150d263f-d8d0-41bc-b04b-394586738282"
-					(reference "R12")
+					(reference "R4")
 					(unit 1)
 				)
@@
 		(dnp no)
 		(fields_autoplaced yes)
-		(property "Reference" "C7"
+		(property "Reference" "C6"
 			(at 69.85 73.6662 0)
 			(show_name no)
@@
 			(project "ROV CTD"
 				(path "/4b85b8a1-3b52-4af9-b3a4-471ab529b035/150d263f-d8d0-41bc-b04b-394586738282"
-					(reference "C7")
+					(reference "C6")
 					(unit 1)
 				)
@@
 		(dnp yes)
 		(fields_autoplaced yes)
-		(property "Reference" "JP3"
+		(property "Reference" "JP1"
 			(at 210.82 91.44 0)
 			(hide yes)
@@
 			(project "ROV CTD"
 				(path "/4b85b8a1-3b52-4af9-b3a4-471ab529b035/150d263f-d8d0-41bc-b04b-394586738282"
-					(reference "JP3")
+					(reference "JP1")
 					(unit 1)
 				)
@@
 		(dnp no)
 		(fields_autoplaced yes)
-		(property "Reference" "#PWR010"
+		(property "Reference" "#PWR025"
 			(at 175.26 72.39 0)
 			(hide yes)
@@
 			(project "ROV CTD"
 				(path "/4b85b8a1-3b52-4af9-b3a4-471ab529b035/150d263f-d8d0-41bc-b04b-394586738282"
-					(reference "#PWR010")
+					(reference "#PWR025")
 					(unit 1)
 				)
@@
 		(dnp no)
 		(fields_autoplaced yes)
-		(property "Reference" "#PWR01"
+		(property "Reference" "#PWR026"
 			(at 190.5 74.93 0)
 			(hide yes)
@@
 			(project "ROV CTD"
 				(path "/4b85b8a1-3b52-4af9-b3a4-471ab529b035/150d263f-d8d0-41bc-b04b-394586738282"
-					(reference "#PWR01")
+					(reference "#PWR026")
 					(unit 1)
 				)
@@
 		(dnp no)
 		(fields_autoplaced yes)
-		(property "Reference" "#PWR07"
+		(property "Reference" "#PWR024"
 			(at 166.37 72.39 0)
 			(hide yes)
@@
 			(project "ROV CTD"
 				(path "/4b85b8a1-3b52-4af9-b3a4-471ab529b035/150d263f-d8d0-41bc-b04b-394586738282"
-					(reference "#PWR07")
+					(reference "#PWR024")
 					(unit 1)
 				)
@@
 		(dnp no)
 		(fields_autoplaced yes)
-		(property "Reference" "#PWR023"
+		(property "Reference" "#PWR020"
 			(at 67.31 73.66 0)
 			(hide yes)
@@
 			(project "ROV CTD"
 				(path "/4b85b8a1-3b52-4af9-b3a4-471ab529b035/150d263f-d8d0-41bc-b04b-394586738282"
-					(reference "#PWR023")
+					(reference "#PWR020")
 					(unit 1)
 				)
@@
 		(dnp no)
 		(fields_autoplaced yes)
-		(property "Reference" "#PWR029"
+		(property "Reference" "#PWR023"
 			(at 67.31 107.95 0)
 			(hide yes)
@@
 			(project "ROV CTD"
 				(path "/4b85b8a1-3b52-4af9-b3a4-471ab529b035/150d263f-d8d0-41bc-b04b-394586738282"
-					(reference "#PWR029")
+					(reference "#PWR023")
 					(unit 1)
 				)
@@
 		(dnp no)
 		(fields_autoplaced yes)
-		(property "Reference" "#PWR022"
+		(property "Reference" "#PWR031"
 			(at 214.63 105.41 0)
 			(hide yes)
@@
 			(project "ROV CTD"
 				(path "/4b85b8a1-3b52-4af9-b3a4-471ab529b035/150d263f-d8d0-41bc-b04b-394586738282"
-					(reference "#PWR022")
+					(reference "#PWR031")
 					(unit 1)
 				)
@@
 		(dnp no)
 		(fields_autoplaced yes)
-		(property "Reference" "#PWR024"
+		(property "Reference" "#PWR021"
 			(at 67.31 86.36 0)
 			(hide yes)
@@
 			(project "ROV CTD"
 				(path "/4b85b8a1-3b52-4af9-b3a4-471ab529b035/150d263f-d8d0-41bc-b04b-394586738282"
-					(reference "#PWR024")
+					(reference "#PWR021")
 					(unit 1)
 				)
@@
 		(dnp no)
 		(fields_autoplaced yes)
-		(property "Reference" "#PWR013"
+		(property "Reference" "#PWR027"
 			(at 190.5 97.79 0)
 			(hide yes)
@@
 			(project "ROV CTD"
 				(path "/4b85b8a1-3b52-4af9-b3a4-471ab529b035/150d263f-d8d0-41bc-b04b-394586738282"
-					(reference "#PWR013")
+					(reference "#PWR027")
 					(unit 1)
 				)
@@
 		(dnp no)
 		(fields_autoplaced yes)
-		(property "Reference" "R14"
+		(property "Reference" "R3"
 			(at 177.8 72.3899 0)
 			(show_name no)
@@
 			(project "ROV CTD"
 				(path "/4b85b8a1-3b52-4af9-b3a4-471ab529b035/150d263f-d8d0-41bc-b04b-394586738282"
-					(reference "R14")
+					(reference "R3")
 					(unit 1)
 				)
@@
 		(dnp yes)
 		(fields_autoplaced yes)
-		(property "Reference" "JP4"
+		(property "Reference" "JP2"
 			(at 219.71 91.44 0)
 			(hide yes)
@@
 			(project "ROV CTD"
 				(path "/4b85b8a1-3b52-4af9-b3a4-471ab529b035/150d263f-d8d0-41bc-b04b-394586738282"
-					(reference "JP4")
+					(reference "JP2")
 					(unit 1)
 				)
@@
 		(dnp no)
 		(fields_autoplaced yes)
-		(property "Reference" "C8"
+		(property "Reference" "C7"
 			(at 69.85 95.2562 0)
 			(show_name no)
@@
 			(project "ROV CTD"
 				(path "/4b85b8a1-3b52-4af9-b3a4-471ab529b035/150d263f-d8d0-41bc-b04b-394586738282"
-					(reference "C8")
+					(reference "C7")
 					(unit 1)
 				)
@@
 		(dnp no)
 		(fields_autoplaced yes)
-		(property "Reference" "#PWR018"
+		(property "Reference" "#PWR029"
 			(at 205.74 105.41 0)
 			(hide yes)
@@
 			(project "ROV CTD"
 				(path "/4b85b8a1-3b52-4af9-b3a4-471ab529b035/150d263f-d8d0-41bc-b04b-394586738282"
-					(reference "#PWR018")
+					(reference "#PWR029")
 					(unit 1)
 				)
@@
 		(dnp no)
 		(fields_autoplaced yes)
-		(property "Reference" "#PWR06"
+		(property "Reference" "#PWR030"
 			(at 214.63 72.39 0)
 			(hide yes)
@@
 			(project "ROV CTD"
 				(path "/4b85b8a1-3b52-4af9-b3a4-471ab529b035/150d263f-d8d0-41bc-b04b-394586738282"
-					(reference "#PWR06")
+					(reference "#PWR030")
 					(unit 1)
 				)
@@
 		(dnp no)
 		(fields_autoplaced yes)
-		(property "Reference" "#PWR03"
+		(property "Reference" "#PWR028"
 			(at 205.74 72.39 0)
 			(hide yes)
@@
 			(project "ROV CTD"
 				(path "/4b85b8a1-3b52-4af9-b3a4-471ab529b035/150d263f-d8d0-41bc-b04b-394586738282"
-					(reference "#PWR03")
+					(reference "#PWR028")
 					(unit 1)
 				)

Commit message: working on CDT
Parts:
- renumbered C6 to C33, C7 to C34, R2 to R30, R3 to R31, R4 to R32, R5 to R33
Changed lines of the file:
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@@
 			(justify left bottom)
 		)
-		(property "Net Class" "PCBway min 1 oz "
+		(property "Netclass" "PCBway min 1 oz "
 			(at 153.0299 104.41 0)
 			(show_name no)
@@
 			(justify left bottom)
 		)
-		(property "Net Class" "PCBway min 1 oz "
+		(property "Netclass" "PCBway min 1 oz "
 			(at 153.0299 101.87 0)
 			(show_name no)
@@
 			(justify left bottom)
 		)
-		(property "Net Class" "PCBway min 1 oz "
+		(property "Netclass" "PCBway min 1 oz "
 			(at 122.5499 104.41 0)
 			(show_name no)
@@
 			(justify left bottom)
 		)
-		(property "Net Class" "PCBway min 1 oz "
+		(property "Netclass" "PCBway min 1 oz "
 			(at 122.5499 101.87 0)
 			(show_name no)
@@
 			(justify left bottom)
 		)
-		(property "Net Class" "PCBway min 1 oz "
+		(property "Netclass" "PCBway min 1 oz "
 			(at 153.0299 99.33 0)
 			(show_name no)
@@
 		(dnp no)
 		(fields_autoplaced yes)
-		(property "Reference" "R2"
+		(property "Reference" "R30"
 			(at 168.91 72.3899 0)
 			(show_name no)
@@
 		(instances
 			(project "ROV CTD"
-				(path "/4b85b8a1-3b52-4af9-b3a4-471ab529b035/150d263f-d8d0-41bc-b04b-394586738282"
-					(reference "R2")
+				(path "/4b85b8a1-3b52-4af9-b3a4-471ab529b035/d2e3d421-56cf-4c4b-84e7-3f0b55169ef2"
+					(reference "R30")
 					(unit 1)
 				)
@@
 		(dnp no)
 		(fields_autoplaced yes)
-		(property "Reference" "#PWR022"
+		(property "Reference" "#PWR0112"
 			(at 67.31 95.25 0)
 			(hide yes)
@@
 		(instances
 			(project "ROV CTD"
-				(path "/4b85b8a1-3b52-4af9-b3a4-471ab529b035/150d263f-d8d0-41bc-b04b-394586738282"
-					(reference "#PWR022")
+				(path "/4b85b8a1-3b52-4af9-b3a4-471ab529b035/d2e3d421-56cf-4c4b-84e7-3f0b55169ef2"
+					(reference "#PWR0112")
 					(unit 1)
 				)
@@
 		(dnp no)
 		(fields_autoplaced yes)
-		(property "Reference" "R5"
+		(property "Reference" "R33"
 			(at 217.17 72.3899 0)
 			(show_name no)
@@
 		(instances
 			(project "ROV CTD"
-				(path "/4b85b8a1-3b52-4af9-b3a4-471ab529b035/150d263f-d8d0-41bc-b04b-394586738282"
-					(reference "R5")
+				(path "/4b85b8a1-3b52-4af9-b3a4-471ab529b035/d2e3d421-56cf-4c4b-84e7-3f0b55169ef2"
+					(reference "R33")
 					(unit 1)
 				)
@@
 		(instances
 			(project "ROV CTD"
-				(path "/4b85b8a1-3b52-4af9-b3a4-471ab529b035/150d263f-d8d0-41bc-b04b-394586738282"
+				(path "/4b85b8a1-3b52-4af9-b3a4-471ab529b035/d2e3d421-56cf-4c4b-84e7-3f0b55169ef2"
 					(reference "M1")
 					(unit 1)
@@
 		(dnp no)
 		(fields_autoplaced yes)
-		(property "Reference" "R4"
+		(property "Reference" "R32"
 			(at 208.28 72.3899 0)
 			(show_name no)
@@
 		(instances
 			(project "ROV CTD"
-				(path "/4b85b8a1-3b52-4af9-b3a4-471ab529b035/150d263f-d8d0-41bc-b04b-394586738282"
-					(reference "R4")
+				(path "/4b85b8a1-3b52-4af9-b3a4-471ab529b035/d2e3d421-56cf-4c4b-84e7-3f0b55169ef2"
+					(reference "R32")
 					(unit 1)
 				)
@@
 		(dnp no)
 		(fields_autoplaced yes)
-		(property "Reference" "C6"
+		(property "Reference" "C33"
 			(at 69.85 73.6662 0)
 			(show_name no)
@@
 		(instances
 			(project "ROV CTD"
-				(path "/4b85b8a1-3b52-4af9-b3a4-471ab529b035/150d263f-d8d0-41bc-b04b-394586738282"
-					(reference "C6")
+				(path "/4b85b8a1-3b52-4af9-b3a4-471ab529b035/d2e3d421-56cf-4c4b-84e7-3f0b55169ef2"
+					(reference "C33")
 					(unit 1)
 				)
@@
 		(instances
 			(project "ROV CTD"
-				(path "/4b85b8a1-3b52-4af9-b3a4-471ab529b035/150d263f-d8d0-41bc-b04b-394586738282"
+				(path "/4b85b8a1-3b52-4af9-b3a4-471ab529b035/d2e3d421-56cf-4c4b-84e7-3f0b55169ef2"
 					(reference "JP1")
 					(unit 1)
@@
 		(dnp no)
 		(fields_autoplaced yes)
-		(property "Reference" "#PWR025"
+		(property "Reference" "#PWR0115"
 			(at 175.26 72.39 0)
 			(hide yes)
@@
 		(instances
 			(project "ROV CTD"
-				(path "/4b85b8a1-3b52-4af9-b3a4-471ab529b035/150d263f-d8d0-41bc-b04b-394586738282"
-					(reference "#PWR025")
+				(path "/4b85b8a1-3b52-4af9-b3a4-471ab529b035/d2e3d421-56cf-4c4b-84e7-3f0b55169ef2"
+					(reference "#PWR0115")
 					(unit 1)
 				)
@@
 		(dnp no)
 		(fields_autoplaced yes)
-		(property "Reference" "#PWR026"
+		(property "Reference" "#PWR0116"
 			(at 190.5 74.93 0)
 			(hide yes)
@@
 		(instances
 			(project "ROV CTD"
-				(path "/4b85b8a1-3b52-4af9-b3a4-471ab529b035/150d263f-d8d0-41bc-b04b-394586738282"
-					(reference "#PWR026")
+				(path "/4b85b8a1-3b52-4af9-b3a4-471ab529b035/d2e3d421-56cf-4c4b-84e7-3f0b55169ef2"
+					(reference "#PWR0116")
 					(unit 1)
 				)
@@
 		(dnp no)
 		(fields_autoplaced yes)
-		(property "Reference" "#PWR024"
+		(property "Reference" "#PWR0114"
 			(at 166.37 72.39 0)
 			(hide yes)
@@
 		(instances
 			(project "ROV CTD"
-				(path "/4b85b8a1-3b52-4af9-b3a4-471ab529b035/150d263f-d8d0-41bc-b04b-394586738282"
-					(reference "#PWR024")
+				(path "/4b85b8a1-3b52-4af9-b3a4-471ab529b035/d2e3d421-56cf-4c4b-84e7-3f0b55169ef2"
+					(reference "#PWR0114")
 					(unit 1)
 				)
@@
 		(dnp no)
 		(fields_autoplaced yes)
-		(property "Reference" "#PWR020"
+		(property "Reference" "#PWR0110"
 			(at 67.31 73.66 0)
 			(hide yes)
@@
 		(instances
 			(project "ROV CTD"
-				(path "/4b85b8a1-3b52-4af9-b3a4-471ab529b035/150d263f-d8d0-41bc-b04b-394586738282"
-					(reference "#PWR020")
+				(path "/4b85b8a1-3b52-4af9-b3a4-471ab529b035/d2e3d421-56cf-4c4b-84e7-3f0b55169ef2"
+					(reference "#PWR0110")
 					(unit 1)
 				)
@@
 		(dnp no)
 		(fields_autoplaced yes)
-		(property "Reference" "#PWR023"
+		(property "Reference" "#PWR0113"
 			(at 67.31 107.95 0)
 			(hide yes)
@@
 		(instances
 			(project "ROV CTD"
-				(path "/4b85b8a1-3b52-4af9-b3a4-471ab529b035/150d263f-d8d0-41bc-b04b-394586738282"
-					(reference "#PWR023")
+				(path "/4b85b8a1-3b52-4af9-b3a4-471ab529b035/d2e3d421-56cf-4c4b-84e7-3f0b55169ef2"
+					(reference "#PWR0113")
 					(unit 1)
 				)
@@
 		(dnp no)
 		(fields_autoplaced yes)
-		(property "Reference" "#PWR031"
+		(property "Reference" "#PWR0121"
 			(at 214.63 105.41 0)
 			(hide yes)
@@
 		(instances
 			(project "ROV CTD"
-				(path "/4b85b8a1-3b52-4af9-b3a4-471ab529b035/150d263f-d8d0-41bc-b04b-394586738282"
-					(reference "#PWR031")
+				(path "/4b85b8a1-3b52-4af9-b3a4-471ab529b035/d2e3d421-56cf-4c4b-84e7-3f0b55169ef2"
+					(reference "#PWR0121")
 					(unit 1)
 				)
@@
 		(dnp no)
 		(fields_autoplaced yes)
-		(property "Reference" "#PWR021"
+		(property "Reference" "#PWR0111"
 			(at 67.31 86.36 0)
 			(hide yes)
@@
 		(instances
 			(project "ROV CTD"
-				(path "/4b85b8a1-3b52-4af9-b3a4-471ab529b035/150d263f-d8d0-41bc-b04b-394586738282"
-					(reference "#PWR021")
+				(path "/4b85b8a1-3b52-4af9-b3a4-471ab529b035/d2e3d421-56cf-4c4b-84e7-3f0b55169ef2"
+					(reference "#PWR0111")
 					(unit 1)
 				)
@@
 		(dnp no)
 		(fields_autoplaced yes)
-		(property "Reference" "#PWR027"
+		(property "Reference" "#PWR0117"
 			(at 190.5 97.79 0)
 			(hide yes)
@@
 		(instances
 			(project "ROV CTD"
-				(path "/4b85b8a1-3b52-4af9-b3a4-471ab529b035/150d263f-d8d0-41bc-b04b-394586738282"
-					(reference "#PWR027")
+				(path "/4b85b8a1-3b52-4af9-b3a4-471ab529b035/d2e3d421-56cf-4c4b-84e7-3f0b55169ef2"
+					(reference "#PWR0117")
 					(unit 1)
 				)
@@
 		(dnp no)
 		(fields_autoplaced yes)
-		(property "Reference" "R3"
+		(property "Reference" "R31"
 			(at 177.8 72.3899 0)
 			(show_name no)
@@
 		(instances
 			(project "ROV CTD"
-				(path "/4b85b8a1-3b52-4af9-b3a4-471ab529b035/150d263f-d8d0-41bc-b04b-394586738282"
-					(reference "R3")
+				(path "/4b85b8a1-3b52-4af9-b3a4-471ab529b035/d2e3d421-56cf-4c4b-84e7-3f0b55169ef2"
+					(reference "R31")
 					(unit 1)
 				)
@@
 		(instances
 			(project "ROV CTD"
-				(path "/4b85b8a1-3b52-4af9-b3a4-471ab529b035/150d263f-d8d0-41bc-b04b-394586738282"
+				(path "/4b85b8a1-3b52-4af9-b3a4-471ab529b035/d2e3d421-56cf-4c4b-84e7-3f0b55169ef2"
 					(reference "JP2")
 					(unit 1)
@@
 		(dnp no)
 		(fields_autoplaced yes)
-		(property "Reference" "C7"
+		(property "Reference" "C34"
 			(at 69.85 95.2562 0)
 			(show_name no)
@@
 		(instances
 			(project "ROV CTD"
-				(path "/4b85b8a1-3b52-4af9-b3a4-471ab529b035/150d263f-d8d0-41bc-b04b-394586738282"
-					(reference "C7")
+				(path "/4b85b8a1-3b52-4af9-b3a4-471ab529b035/d2e3d421-56cf-4c4b-84e7-3f0b55169ef2"
+					(reference "C34")
 					(unit 1)
 				)
@@
 		(dnp no)
 		(fields_autoplaced yes)
-		(property "Reference" "#PWR029"
+		(property "Reference" "#PWR0119"
 			(at 205.74 105.41 0)
 			(hide yes)
@@
 		(instances
 			(project "ROV CTD"
-				(path "/4b85b8a1-3b52-4af9-b3a4-471ab529b035/150d263f-d8d0-41bc-b04b-394586738282"
-					(reference "#PWR029")
+				(path "/4b85b8a1-3b52-4af9-b3a4-471ab529b035/d2e3d421-56cf-4c4b-84e7-3f0b55169ef2"
+					(reference "#PWR0119")
 					(unit 1)
 				)
@@
 		(dnp no)
 		(fields_autoplaced yes)
-		(property "Reference" "#PWR030"
+		(property "Reference" "#PWR0120"
 			(at 214.63 72.39 0)
 			(hide yes)
@@
 		(instances
 			(project "ROV CTD"
-				(path "/4b85b8a1-3b52-4af9-b3a4-471ab529b035/150d263f-d8d0-41bc-b04b-394586738282"
-					(reference "#PWR030")
+				(path "/4b85b8a1-3b52-4af9-b3a4-471ab529b035/d2e3d421-56cf-4c4b-84e7-3f0b55169ef2"
+					(reference "#PWR0120")
 					(unit 1)
 				)
@@
 		(dnp no)
 		(fields_autoplaced yes)
-		(property "Reference" "#PWR028"
+		(property "Reference" "#PWR0118"
 			(at 205.74 72.39 0)
 			(hide yes)
@@
 		(instances
 			(project "ROV CTD"
-				(path "/4b85b8a1-3b52-4af9-b3a4-471ab529b035/150d263f-d8d0-41bc-b04b-394586738282"
-					(reference "#PWR028")
-					(unit 1)
-				)
+				(path "/4b85b8a1-3b52-4af9-b3a4-471ab529b035/d2e3d421-56cf-4c4b-84e7-3f0b55169ef2"
+					(reference "#PWR0118")
+					(unit 1)
+				)
