File: ROV - Conductivity Temperature and Depth Transducer/KiCAD/ROV CTD_old.kicad_sch (KiCad schematic)
At the start: 20 parts, among them J2 Temp, J4 Conn_02x06_Odd_Even, J5 Conn_02x05_Odd_Even, J7 Conn_02x06_Odd_Even, J8 Conn_02x06_Odd_Even, U4 RT9166/A

Commit message: working on CDT
Parts:
- removed C19, C6: 10nF, Capacitor_SMD:C_0805_2012Metric_Pad1.18x1.45mm_HandSolder, symbol Device:C_Small
- removed C20, C7: 100nF, Capacitor_SMD:C_0805_2012Metric_Pad1.18x1.45mm_HandSolder, symbol Device:C_Small
- removed D12: Status_Led, LED_SMD:LED_0805_2012Metric_Pad1.15x1.40mm_HandSolder, symbol Device:LED_Small_Filled
- removed J2: Temp, Connector_PinHeader_1.00mm:PinHeader_1x02_P1.00mm_Vertical, symbol Connector_Generic:Conn_01x02
- removed J4: Conn_02x06_Odd_Even, Connector_PinSocket_1.27mm:PinSocket_2x06_P1.27mm_Vertical_SMD, symbol Connector_Generic:Conn_02x06_Odd_Even
- removed J7, J8: Conn_02x06_Odd_Even, Connector_PinHeader_1.27mm:PinHeader_2x06_P1.27mm_Vertical_SMD, symbol Connector_Generic:Conn_02x06_Odd_Even
- removed R15: 4k7, Resistor_SMD:R_0805_2012Metric_Pad1.20x1.40mm_HandSolder, symbol Device:R_Small
- removed R16, R17, R18: 470, Resistor_SMD:R_0805_2012Metric_Pad1.20x1.40mm_HandSolder, symbol Device:R_Small
- removed R5: 10k, Resistor_SMD:R_0805_2012Metric_Pad1.20x1.40mm_HandSolder, symbol Device:R_Small
- removed U4: RT9166/A, Package_TO_SOT_SMD:SOT-23_Handsoldering, symbol KiCad Symbols:RT9166/A
- added C2, C4: 10nF, Capacitor_SMD:C_0805_2012Metric_Pad1.18x1.45mm_HandSolder, symbol Device:C_Small
- added C3, C5: 100nF, Capacitor_SMD:C_0805_2012Metric_Pad1.18x1.45mm_HandSolder, symbol Device:C_Small
- added D7: Status_Led, LED_SMD:LED_0805_2012Metric_Pad1.15x1.40mm_HandSolder, symbol Device:LED_Small_Filled
- added J1: Temp, Connector_PinHeader_1.00mm:PinHeader_1x02_P1.00mm_Vertical, symbol Connector_Generic:Conn_01x02
- added J2: Conn_02x05_Odd_Even, Connector_PinSocket_1.27mm:PinSocket_2x05_P1.27mm_Vertical_SMD, symbol Connector_Generic:Conn_02x05_Odd_Even
- added J3, J4: Conn_02x05_Odd_Even, Connector_PinHeader_1.27mm:PinHeader_2x05_P1.27mm_Vertical_SMD, symbol Connector_Generic:Conn_02x05_Odd_Even
- added R1: 10k, Resistor_SMD:R_0805_2012Metric_Pad1.20x1.40mm_HandSolder, symbol Device:R_Small
- added U1: RT9166/A, Package_TO_SOT_SMD:SOT-23_Handsoldering, symbol KiCad Symbols:RT9166/A
- J5: footprint Connector_PinHeader_1.27mm:PinHeader_2x05_P1.27mm_Vertical_SMD -> Connector_PinSocket_1.27mm:PinSocket_2x05_P1.27mm_Vertical_SMD
Connections:
- net +3V3: now also C3.1, C4.1, U1.2 (OUT)
- net +5V: now also J2.3 (Pin_3)
- net +5V_Bot: now also C2.1, J4.3 (Pin_3), R1.2, U1.3 (IN); no longer J5.3 (Pin_3)
- net +5V_Mid: now also J5.3 (Pin_3), J3.3 (Pin_3)
- net Bot_Probe_1: now also J4.5 (Pin_5); no longer J5.5 (Pin_5)
- net Bot_Probe_2: now also J4.6 (Pin_6); no longer J5.6 (Pin_6)
- net Bot_SCL: now also J4.8 (Pin_8); no longer J5.8 (Pin_8)
- net Bot_SDA: now also J4.10 (Pin_10); no longer J5.10 (Pin_10)
- net Bot_Status_LED: now also J4.9 (Pin_9); no longer J5.9 (Pin_9)
- net Bot_Temp: now also C5.1, J1.2 (Pin_2), J4.7 (Pin_7), R1.1; no longer J5.7 (Pin_7)
- net GND: now also C2.2, C3.2, C4.2, C5.2, D7.1 (K), J1.1 (Pin_1), J2.2 (Pin_2), J2.4 (Pin_4), J3.2 (Pin_2), J3.4 (Pin_4), J4.2 (Pin_2), J4.4 (Pin_4), U1.1 (GND)
- net Mid_Probe_1: now also J5.5 (Pin_5)
- net Mid_Probe_2: now also J5.6 (Pin_6)
- net Mid_SCL: now also J5.8 (Pin_8), J3.8 (Pin_8)
- net Mid_SDA: now also J5.10 (Pin_10), J3.10 (Pin_10)
- net Mid_Status_LED: now also J5.9 (Pin_9), J3.9 (Pin_9)
- net Mid_TDS: now also J3.6 (Pin_6)
- net Mid_TDS_OSC: now also J3.7 (Pin_7)
- net Mid_Temp: now also J5.7 (Pin_7), J3.5 (Pin_5)
- net SCL: now also J2.8 (Pin_8)
- net SDA: now also J2.10 (Pin_10)
- net STATUS_LED: now also J2.9 (Pin_9)
- net Top_TDS: now also J2.6 (Pin_6)
- net Top_TDS_OSC: now also J2.7 (Pin_7)
- net Top_Temp: now also J2.5 (Pin_5)
- net V_in: now also J2.1 (Pin_1)
- net at R21.2: now also D7.2 (A)
- no-connect marks 6 -> 4
Other:
- title: ROV Light Module -> ROV CTD
