File: ROV - Conductivity Temperature and Depth Transducer/KiCAD/ROV CTD.kicad_pcb (KiCad board)
At the start: 2 copper layers, 73.7 x 23.4 mm, 79 parts, among them J2 Temp, J4 Bottom - Middle, J6 Main In, J7 Bottom - Middle, J8 Middle - Top, J9 Top - Middle, M2 MS5803-14BA, U1 LMV324, U2 ATtiny1614-Arduino, U3 AP63205WU, U4 LM2664, U5 RT9166/A, U6 MAX3072E

Commit message: massive cleanup
Parts:
- removed C28: 1uF, Capacitor_SMD:C_0805_2012Metric_Pad1.18x1.45mm_HandSolder
- removed C29, C30: 100nF, Capacitor_SMD:C_0805_2012Metric_Pad1.18x1.45mm_HandSolder
- removed C31, C32: 10nF, Capacitor_SMD:C_0805_2012Metric_Pad1.18x1.45mm_HandSolder
- removed D10: 5V, LED_SMD:LED_0805_2012Metric_Pad1.15x1.40mm_HandSolder
- removed D9: 1N4148WT, Diode_SMD:D_SOD-523
- removed J8: Middle - Top, Connector_PinSocket_1.27mm:PinSocket_2x06_P1.27mm_Vertical_SMD
- removed J9: Top - Middle, Connector_PinHeader_1.27mm:PinHeader_2x06_P1.27mm_Vertical_SMD
- removed JP3, JP4: RX, Jumper:SolderJumper-2_P1.3mm_Open_TrianglePad1.0x1.5mm
- removed L2: 4.7uH, Inductor_SMD:L_Vishay_IHLP-1212
- removed M2: MS5803-14BA, KiCad Footprints:MS5803-14BA
- removed R21, R22, R23, R27, R28: 36k, Resistor_SMD:R_0805_2012Metric_Pad1.20x1.40mm_HandSolder
- removed R24, R25: 10k, Resistor_SMD:R_0805_2012Metric_Pad1.20x1.40mm_HandSolder
- removed R26: 1k, Resistor_SMD:R_0805_2012Metric_Pad1.20x1.40mm_HandSolder
- added C1: 100nF, Capacitor_SMD:C_0805_2012Metric_Pad1.18x1.45mm_HandSolder, F.Cu at (141.1, 136.4)
- added C2: 10nF, Capacitor_SMD:C_0805_2012Metric_Pad1.18x1.45mm_HandSolder, F.Cu at (141.1, 139.4)
- added D3: 1N4148WT, Diode_SMD:D_SOD-523, F.Cu at (137.5, 146.5)
- added D6: Power, LED_SMD:LED_0805_2012Metric_Pad1.15x1.40mm_HandSolder, F.Cu at (143.7, 151.4)
- added J1: Temp, Connector_PinHeader_1.00mm:PinHeader_1x02_P1.00mm_Vertical, F.Cu at (142.2, 131.0)
- added J3: Conn_02x05_Odd_Even, Connector_PinHeader_1.27mm:PinHeader_2x05_P1.27mm_Vertical_SMD, F.Cu at (135.8, 130.7)
- added J5: Conn_02x05_Odd_Even, Connector_PinSocket_1.27mm:PinSocket_2x05_P1.27mm_Vertical_SMD, F.Cu at (134.8, 139.1)
- added L1: 4.7uH, Inductor_SMD:L_Vishay_IHLP-1212, F.Cu at (144.2, 147.6)
- added R1: 10k, Resistor_SMD:R_0805_2012Metric_Pad1.20x1.40mm_HandSolder, F.Cu at (142.9, 128.0)
- added R16: 10k, Resistor_SMD:R_0805_2012Metric_Pad1.20x1.40mm_HandSolder, F.Cu at (133.3, 152.7)
- added R2: 2k2, Resistor_SMD:R_0805_2012Metric_Pad1.20x1.40mm_HandSolder, F.Cu at (149.7, 128.0)
- added R3: 2k2, Resistor_SMD:R_0805_2012Metric_Pad1.20x1.40mm_HandSolder, F.Cu at (149.7, 130.9)
- added R4: 10k, Resistor_SMD:R_0805_2012Metric_Pad1.20x1.40mm_HandSolder, F.Cu at (149.7, 133.9)
- added R5: 10k, Resistor_SMD:R_0805_2012Metric_Pad1.20x1.40mm_HandSolder, F.Cu at (149.7, 136.8)
- added R6: 51k, Resistor_SMD:R_0805_2012Metric_Pad1.20x1.40mm_HandSolder, F.Cu at (133.3, 146.8)
- added R8: 1k, Resistor_SMD:R_0805_2012Metric_Pad1.20x1.40mm_HandSolder, F.Cu at (133.3, 149.7)
- C10: value 47uF -> 100uF
- C11: value 100uF -> 1uF
- C14: value 10uF -> 1uF
- C15: value 100nF -> 4.7uF
- C16: value 22uF -> 100nF
- C17: value 22uF -> 4.7uF
- C18: value 10uF -> 100nF
- C19: value 100nF -> 20pF
- C20: value 100nF -> 10pF
- C22: value 20pF -> 10uF
- C23: value 4.7uF -> 100nF
- C24: value 100nF -> 22uF
- C25: value 4.7uF -> 22uF
- C26: value 100nF -> 47uF
- C27: value 1uF -> 10pF
- C4: value 10pF -> 10nF
- C6: value 10pF -> 100nF
- C7: value 100nF -> 10nF
- C8: value 10nF -> 10uF
- C9: value 47uF -> 100nF
- D4: value Status -> CZRB5370B-HF; footprint LED_SMD:LED_0805_2012Metric_Pad1.15x1.40mm_HandSolder -> Diode_SMD:D_SMB_Handsoldering
- D5: value CZRB5370B-HF -> Status; footprint Diode_SMD:D_SMB_Handsoldering -> LED_SMD:LED_0805_2012Metric_Pad1.15x1.40mm_HandSolder
- J2: value Temp -> Conn_02x05_Odd_Even; footprint Connector_PinHeader_1.00mm:PinHeader_1x02_P1.00mm_Vertical -> Connector_PinSocket_1.27mm:PinSocket_2x05_P1.27mm_Vertical_SMD
- J4: value Bottom - Middle -> Conn_02x05_Odd_Even; footprint Connector_PinSocket_1.27mm:PinSocket_2x06_P1.27mm_Vertical_SMD -> Connector_PinHeader_1.27mm:PinHeader_2x05_P1.27mm_Vertical_SMD
- J6: footprint Connector_PinHeader_2.54mm:PinHeader_1x05_P2.54mm_Vertical -> Connector_PinHeader_2.54mm:PinHeader_1x05_P2.54mm_Vertical_SMD_Pin1Left; moved to B.Cu
- J7: value Bottom - Middle -> AVR UPDI Header; footprint Connector_PinHeader_1.27mm:PinHeader_2x06_P1.27mm_Vertical_SMD -> Connector_PinHeader_1.27mm:PinHeader_2x03_P1.27mm_Vertical_SMD
- JP1: value TX -> RX
- R10: value 12k -> 820
- R11: value 1k -> 36k
- R12, R13: value 10k -> 36k
- R14, R15: value 2k2 -> 36k
- R17: value 2k -> 51k
- R18: value 51k -> 12k
- R19: value 1M -> 520
- R20: value 820 -> 470
- R7: value 520 -> 2k
- R9: value 37k -> 1M
- U1: value LMV324 -> RT9166/A; footprint Package_SO:SOIC-14_3.9x8.7mm_P1.27mm -> Package_TO_SOT_SMD:SOT-23_Handsoldering
- U2: value ATtiny1614-Arduino -> LM2664; footprint Package_SO:SOIC-14_3.9x8.7mm_P1.27mm -> Package_TO_SOT_SMD:SOT-23-6
- U3: value AP63205WU -> LMV324; footprint Package_TO_SOT_SMD:TSOT-23-6 -> Package_SO:SOIC-14_3.9x8.7mm_P1.27mm
- U4: value LM2664 -> ATtiny1614-Arduino; footprint Package_TO_SOT_SMD:SOT-23-6 -> Package_SO:SOIC-14_3.9x8.7mm_P1.27mm
- U5: value RT9166/A -> AP63205WU; footprint Package_TO_SOT_SMD:SOT-23_Handsoldering -> Package_TO_SOT_SMD:TSOT-23-6
- U6: value MAX3072E -> MAX13487E
- moved J6 5.08 mm to (190.5, 115.2), turned to -90 degrees
- moved U5 3.30 mm to (136.5, 106.0)
- moved J2 1.55 mm to (131.4, 106.0)
Connections:
- C10 pad 1: +5V -> Net-(U2-C_{FLY+})
- C10 pad 2: GND -> Net-(U2-C_{FLY-})
- C11 pad 1: Net-(U4-C_{FLY+}) -> Net-(C11-Pad1)
- C11 pad 2: Net-(U4-C_{FLY-}) -> /Mid_Probe_1
- C13 pad 1: /Vmeasure -> -5V
- C14 pad 1: GND -> /Mid_Probe_2
- C14 pad 2: V_in -> Net-(U3B--)
- C15 pad 1: Net-(U3-SW) -> +5V_Mid
- C15 pad 2: Net-(U3-BST) -> GND
- C16 pad 1: GND -> +5V_Mid
- C16 pad 2: +5V -> GND
- C17 pad 1: GND -> -5V
- C17 pad 2: +5V -> GND
- C18 pad 1: +5V -> -5V
- C19 pad 1: +5V -> /Mid_TDS
- C20 pad 1: -5V -> +5V
- C21 pad 1: /Bot_Temp -> /Arduino Driver PCB/Vmeasure
- C22 pad 1: /Mid_TDS -> GND
- C22 pad 2: GND -> V_in
- C23 pad 1: +5V -> Net-(U5-SW)
- C23 pad 2: GND -> Net-(U5-BST)
- C24 pad 1: +5V -> GND
- C24 pad 2: GND -> +5V
- C25 pad 1: -5V -> GND
- C25 pad 2: GND -> +5V
- C26 pad 1: -5V -> +5V
- C27 pad 1: Net-(C27-Pad1) -> +5V
- C27 pad 2: /Mid_Probe_1 -> GND
- C3 pad 1: +5V -> +3V3
- C4 pad 1: +5V -> +3V3
- C5 pad 1: +5V -> /Bot_Temp
- C6 pad 1: +5V -> +3V3
- C8 pad 1: +3V3 -> +5V_Mid
- C9 pad 1: +5V -> +5V_Mid
- D4 pad 1: GND -> V_in
- D4 pad 2: Net-(D4-A) -> V_Supply
- D5 pad 1: V_in -> GND
- H1 pad 1: /Bot_Probe_1 -> /Bot_Probe_2
- H2 pad 1: /Bot_Probe_2 -> /Bot_Probe_1
- J2 pad 1: GND -> V_in
- J2 pad 2: /Bot_Temp -> GND
- J4 pad 10: GND -> /Bot_SDA
- J4 pad 3: +5V -> +5V_Bot
- J4 pad 5: /Bot_Temp -> /Bot_Probe_1
- J4 pad 6: /Bot_SCL -> /Bot_Probe_2
- J4 pad 7: unconnected-(J4-Pin_7-Pad7) -> /Bot_Temp
- J4 pad 8: /Bot_SDA -> /Bot_SCL
- J4 pad 9: GND -> /Bot_Status_LED
- J6 pad 1: Net-(D5-A) -> V_Supply
- J6 pad 2: /UPDI -> /Arduino Driver PCB/UPDI
- J6 pad 3: /Data_A -> /Arduino Driver PCB/Data_B
- J6 pad 4: /Data_B -> /Arduino Driver PCB/Data_A
- J7 pad 1: unconnected-(J7-Pin_1-Pad1) -> /Arduino Driver PCB/UPDI
- J7 pad 2: GND -> +5V
- J7 pad 3: +5V -> /Arduino Driver PCB/Builtin_LED
- J7 pad 4: GND -> /Arduino Driver PCB/SERIAL_TX
- J7 pad 5: /Mid_Temp -> /Arduino Driver PCB/SERIAL_RX
- J7 pad 6: /Mid_SCL -> GND
- JP1 pad 1: /SERIAL_TX -> GND
- JP1 pad 2: /Data_A -> /Pressure Transducer/PS
- JP2 pad 1: /SERIAL_RX -> GND
- JP2 pad 2: /Data_B -> /Pressure Transducer/AD/CS
- R10 pad 1: /Vmeasure -> Net-(U3B--)
- R10 pad 2: GND -> Net-(R10-Pad2)
- R11 pad 1: +5V -> Net-(R10-Pad2)
- R11 pad 2: Net-(D10-A) -> Net-(U3C--)
- R12 pad 1: +3V3 -> Net-(U3C--)
- R12 pad 2: /Pressure Transducer/PS -> Net-(D2-K)
- R13 pad 1: +3V3 -> Net-(U3C--)
- R13 pad 2: /Pressure Transducer/AD/CS -> Net-(D1-A)
- R14 pad 1: +3V3 -> Net-(D1-A)
- R14 pad 2: /Bot_SDA -> Net-(U3D--)
- R15 pad 1: +3V3 -> Net-(U3D--)
- R15 pad 2: /Bot_SCL -> Net-(R15-Pad2)
- R17 pad 1: Net-(U1A--) -> V_in
- R17 pad 2: Net-(C27-Pad1) -> /Arduino Driver PCB/Vmeasure
- R18 pad 1: /Conductivity Transducer/Osc -> /Arduino Driver PCB/Vmeasure
- R18 pad 2: Net-(U1A--) -> GND
- R19 pad 1: GND -> /Arduino Driver PCB/Builtin_LED
- R19 pad 2: Net-(U1B--) -> Net-(D5-A)
- R20 pad 1: Net-(U1B--) -> +5V
- R20 pad 2: Net-(R20-Pad2) -> Net-(D6-A)
- R7 pad 1: /Builtin_LED -> Net-(U3A--)
- R7 pad 2: Net-(D4-A) -> Net-(C11-Pad1)
- R9 pad 1: V_in -> GND
- R9 pad 2: /Vmeasure -> Net-(U3B--)
- U1 pad 1: Net-(C27-Pad1) -> GND
- U1 pad 2: Net-(U1A--) -> +3V3
- U1 pad 3: GND -> +5V_Bot
- U2 pad 1: +5V -> GND
- U2 pad 2: /A0/D0 -> -5V
- U2 pad 3: /A1/D1 -> Net-(U2-C_{FLY-})
- U2 pad 4: /Builtin_LED -> +5V_Mid
- U2 pad 5: /SERIAL_DIR -> +5V_Mid
- U2 pad 6: /SERIAL_RX -> Net-(U2-C_{FLY+})
- U3 pad 1: +5V -> Net-(C11-Pad1)
- U3 pad 2: V_in -> Net-(U3A--)
- U3 pad 3: V_in -> GND
- U3 pad 4: GND -> +5V_Mid
- U3 pad 5: Net-(U3-SW) -> GND
- U3 pad 6: Net-(U3-BST) -> Net-(U3B--)
- U4 pad 1: GND -> +5V
- U4 pad 2: -5V -> /Top_TDS
- U4 pad 3: Net-(U4-C_{FLY-}) -> /STATUS_LED
- U4 pad 4: +5V -> /Arduino Driver PCB/Builtin_LED
- U4 pad 5: +5V -> /Arduino Driver PCB/A3/D3
- U4 pad 6: Net-(U4-C_{FLY+}) -> /Arduino Driver PCB/SERIAL_RX
- U5 pad 1: GND -> +5V
- U5 pad 2: +3V3 -> V_in
- U5 pad 3: +5V -> V_in
- U6 pad 1: /SERIAL_TX -> /Arduino Driver PCB/SERIAL_RX
- U6 pad 2: /SERIAL_DIR -> +5V
- U6 pad 3: /SERIAL_DIR -> +5V
- U6 pad 4: /SERIAL_RX -> /Arduino Driver PCB/SERIAL_TX
- U6 pad 6: /Data_A -> /Arduino Driver PCB/Data_A
- U6 pad 7: /Data_B -> /Arduino Driver PCB/Data_B
Routing:
- net (no net): track 0.00 -> 67.5 mm, vias 0 -> 2
- net GND: track 21.4 -> 41.9 mm, vias 10 -> 8
- net Net-(U1B--): track 18.0 -> 0.00 mm, vias 1 -> 0
- net /Bot_Temp: track 17.5 -> 0.00 mm, vias 2 -> 0
- net /Arduino Driver PCB/Vmeasure: track 0.00 -> 17.5 mm, vias 0 -> 2
- net /Bot_SCL: track 15.3 -> 0.00 mm, vias 1 -> 0
- net /Bot_SDA: track 15.2 -> 0.00 mm, vias 1 -> 0
- net Net-(C27-Pad1): track 14.3 -> 0.00 mm, vias 1 -> 0
- net Net-(R15-Pad2): track 0.00 -> 13.3 mm, vias 0 -> 1
- net Net-(U3D--): track 0.00 -> 13.2 mm, vias 0 -> 1
- net Net-(D2-K): track 14.4 -> 26.9 mm, vias 0 -> 1
- net /Pressure Transducer/PS: track 12.5 -> 0.00 mm, vias 1 -> 0
- net Net-(U1D--): track 12.5 -> 0.00 mm
- net Net-(U1C--): track 12.2 -> 0.00 mm, vias 2 -> 0
- net /Mid_TDS: track 11.8 -> 0.00 mm
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
Commit message: working on CDT
Parts:
- removed C10: 100uF, Capacitor_SMD:C_0805_2012Metric_Pad1.18x1.45mm_HandSolder
- removed C11: 1uF, Capacitor_SMD:C_0805_2012Metric_Pad1.18x1.45mm_HandSolder
- removed C12, C8: 10uF, Capacitor_SMD:C_0805_2012Metric_Pad1.18x1.45mm_HandSolder
- removed C18, C5: 100nF, Capacitor_SMD:C_0805_2012Metric_Pad1.18x1.45mm_HandSolder
- removed C2: 10nF, Capacitor_SMD:C_0805_2012Metric_Pad1.18x1.45mm_HandSolder
- removed D1, D3: 1N4148WT, Diode_SMD:D_SOD-523
- removed D6: Power, LED_SMD:LED_0805_2012Metric_Pad1.15x1.40mm_HandSolder
- removed J3: Conn_02x05_Odd_Even, Connector_PinHeader_1.27mm:PinHeader_2x05_P1.27mm_Vertical_SMD
- removed L1: 4.7uH, Inductor_SMD:L_Vishay_IHLP-1212
- removed R1, R4: 10k, Resistor_SMD:R_0805_2012Metric_Pad1.20x1.40mm_HandSolder
- removed R12, R13, R14: 36k, Resistor_SMD:R_0805_2012Metric_Pad1.20x1.40mm_HandSolder
- removed R2, R3: 2k2, Resistor_SMD:R_0805_2012Metric_Pad1.20x1.40mm_HandSolder
- removed R8: 1k, Resistor_SMD:R_0805_2012Metric_Pad1.20x1.40mm_HandSolder
- removed the REF** at (153.7, 106.0)
- removed the REF** at (179.1, 106.0)
- removed U1: RT9166/A, Package_TO_SOT_SMD:SOT-23_Handsoldering
- added C28: 4.7uF, Capacitor_SMD:C_0805_2012Metric_Pad1.18x1.45mm_HandSolder, B.Cu at (167.6, 69.2)
- added C29: 100nF, Capacitor_SMD:C_0805_2012Metric_Pad1.18x1.45mm_HandSolder, B.Cu at (167.6, 66.7)
- added C30: 100nF, Capacitor_SMD:C_0805_2012Metric_Pad1.18x1.45mm_HandSolder, B.Cu at (162.6, 74.3)
- added C32: 20pF, Capacitor_SMD:C_0805_2012Metric_Pad1.18x1.45mm_HandSolder, F.Cu at (158.1, 74.0)
- added C33: 100nF, Capacitor_SMD:C_0805_2012Metric_Pad1.18x1.45mm_HandSolder, F.Cu at (104.2, 97.3)
- added C34: 10nF, Capacitor_SMD:C_0805_2012Metric_Pad1.18x1.45mm_HandSolder, F.Cu at (104.2, 100.3)
- added D10: Power, LED_SMD:LED_0805_2012Metric_Pad1.15x1.40mm_HandSolder, B.Cu at (184.2, 83.2)
- added D12: Status_Led, LED_SMD:LED_0805_2012Metric_Pad1.15x1.40mm_HandSolder, F.Cu at (139.7, 83.9)
- added D13: 1N4148WT, Diode_SMD:D_SOD-523, F.Cu at (165.1, 70.2)
- added D14: 1N4148WT, Diode_SMD:D_SOD-523, F.Cu at (158.1, 75.8)
- added J8: Conn_02x06_Odd_Even, Connector_PinHeader_1.27mm:PinHeader_2x06_P1.27mm_Vertical_SMD, F.Cu at (165.1, 83.8)
- added L2: 4.7uH, Inductor_SMD:L_Vishay_IHLP-1212, B.Cu at (191.8, 76.2)
- added R21: 1k, Resistor_SMD:R_0805_2012Metric_Pad1.20x1.40mm_HandSolder, F.Cu at (135.8, 83.9)
- added R22: 1M, Resistor_SMD:R_0805_2012Metric_Pad1.20x1.40mm_HandSolder, F.Cu at (172.2, 79.5)
- added R23: 820, Resistor_SMD:R_0805_2012Metric_Pad1.20x1.40mm_HandSolder, F.Cu at (172.2, 77.5)
- added R24: 36k, Resistor_SMD:R_0805_2012Metric_Pad1.20x1.40mm_HandSolder, F.Cu at (172.2, 75.4)
- added R25: 36k, Resistor_SMD:R_0805_2012Metric_Pad1.20x1.40mm_HandSolder, F.Cu at (168.3, 67.3)
- added R26: 36k, Resistor_SMD:R_0805_2012Metric_Pad1.20x1.40mm_HandSolder, F.Cu at (172.2, 73.4)
- added R27: 36k, Resistor_SMD:R_0805_2012Metric_Pad1.20x1.40mm_HandSolder, F.Cu at (171.8, 69.8)
- added R28: 36k, Resistor_SMD:R_0805_2012Metric_Pad1.20x1.40mm_HandSolder, F.Cu at (158.5, 70.0)
- added R29: 10k, Resistor_SMD:R_0805_2012Metric_Pad1.20x1.40mm_HandSolder, F.Cu at (158.1, 72.0)
- added R30: 2k2, Resistor_SMD:R_0805_2012Metric_Pad1.20x1.40mm_HandSolder, F.Cu at (99.4, 90.2)
- added R31: 2k2, Resistor_SMD:R_0805_2012Metric_Pad1.20x1.40mm_HandSolder, F.Cu at (99.4, 93.2)
- added R32: 10k, Resistor_SMD:R_0805_2012Metric_Pad1.20x1.40mm_HandSolder, F.Cu at (99.4, 96.1)
- added R33: 10k, Resistor_SMD:R_0805_2012Metric_Pad1.20x1.40mm_HandSolder, F.Cu at (99.4, 99.1)
- added REF**: MouseBite-Slot_2.54x2.54mm_on-edge_D0.5mm_P0.85mm_4h_Trace, KiCad Footprints:MouseBite Slot 2.54 x 2.54mm, F.Cu at (179.1, 76.2)
- added REF**: MouseBite-Slot_2.54x2.54mm_on-edge_D0.5mm_P0.85mm_4h_Trace, KiCad Footprints:MouseBite Slot 2.54 x 2.54mm, F.Cu at (153.7, 76.2)
- added U7: LMV324, Package_SO:SOIC-14_3.9x8.7mm_P1.27mm, F.Cu at (165.1, 74.9)
- C1, C13, R5: moved to B.Cu
- C14: value 1uF -> 10uF; moved to B.Cu
- C15: value 4.7uF -> 100nF; moved to B.Cu
- C16: value 100nF -> 22uF; moved to B.Cu
- C17: value 4.7uF -> 22uF; moved to B.Cu
- C19: value 20pF -> 10nF
- C20: value 10pF -> 100nF
- C21: value 100nF -> 10uF; moved to B.Cu
- C22: value 10uF -> 100nF; moved to B.Cu
- C23: value 100nF -> 100uF
- C24: value 22uF -> 1uF
- C25: value 22uF -> 10uF; moved to B.Cu
- C26: value 47uF -> 100nF; moved to B.Cu
- C27: value 10pF -> 1uF; moved to F.Cu
- C3: value 100nF -> 10pF
- C4: value 10nF -> 10pF
- C6: value 100nF -> 10nF; moved to B.Cu
- C7: value 10nF -> 100nF
- C9: value 100nF -> 47uF; moved to B.Cu
- D4: value CZRB5370B-HF -> Status; footprint Diode_SMD:D_SMB_Handsoldering -> LED_SMD:LED_0805_2012Metric_Pad1.15x1.40mm_HandSolder; moved to B.Cu
- D5: value Status -> CZRB5370B-HF; footprint LED_SMD:LED_0805_2012Metric_Pad1.15x1.40mm_HandSolder -> Diode_SMD:D_SMB_Handsoldering; moved to B.Cu
- J1: value Temp -> AVR UPDI Header; footprint Connector_PinHeader_1.00mm:PinHeader_1x02_P1.00mm_Vertical -> Connector_PinHeader_1.27mm:PinHeader_2x03_P1.27mm_Vertical_SMD; moved to B.Cu
- J2: value Conn_02x05_Odd_Even -> Temp; footprint Connector_PinSocket_1.27mm:PinSocket_2x05_P1.27mm_Vertical_SMD -> Connector_PinHeader_1.00mm:PinHeader_1x02_P1.00mm_Vertical; moved to F.Cu
- J4: value Conn_02x05_Odd_Even -> Conn_02x06_Odd_Even; footprint Connector_PinHeader_1.27mm:PinHeader_2x05_P1.27mm_Vertical_SMD -> Connector_PinSocket_1.27mm:PinSocket_2x06_P1.27mm_Vertical_SMD
- J5: footprint Connector_PinSocket_1.27mm:PinSocket_2x05_P1.27mm_Vertical_SMD -> Connector_PinHeader_1.27mm:PinHeader_2x05_P1.27mm_Vertical_SMD; moved to B.Cu
- J7: value AVR UPDI Header -> Conn_02x06_Odd_Even; footprint Connector_PinHeader_1.27mm:PinHeader_2x03_P1.27mm_Vertical_SMD -> Connector_PinHeader_1.27mm:PinHeader_2x06_P1.27mm_Vertical_SMD
- R10: value 820 -> 12k; moved to B.Cu
- R11: value 36k -> 470; moved to B.Cu
- R15: value 36k -> 4k7; moved to B.Cu
- R16: value 10k -> 470; moved to B.Cu
- R17: value 51k -> 470; moved to B.Cu
- R18: value 12k -> 470; moved to B.Cu
- R19: value 520 -> 2k
- R20: value 470 -> 1k
- R7: value 2k -> 520; moved to B.Cu
- R9: value 1M -> 51k; moved to B.Cu
- U2: value LM2664 -> ATtiny1614-Arduino; footprint Package_TO_SOT_SMD:SOT-23-6 -> Package_SO:SOIC-14_3.9x8.7mm_P1.27mm
- U3: value LMV324 -> AP63205WU; footprint Package_SO:SOIC-14_3.9x8.7mm_P1.27mm -> Package_TO_SOT_SMD:TSOT-23-6; moved to B.Cu
- U4: value ATtiny1614-Arduino -> RT9166/A; footprint Package_SO:SOIC-14_3.9x8.7mm_P1.27mm -> Package_TO_SOT_SMD:SOT-23_Handsoldering
- U5: value AP63205WU -> LM2664; footprint Package_TO_SOT_SMD:TSOT-23-6 -> Package_TO_SOT_SMD:SOT-23-6
- moved JP1 108.3 mm to (104.0, 90.5)
- moved JP2 108.3 mm to (104.0, 94.1)
- moved R16 81.9 mm to (162.6, 76.2), turned to 180 degrees
- moved U6 71.3 mm to (184.8, 73.0), turned to 90 degrees
- moved R6 69.8 mm to (158.1, 81.5), turned to 180 degrees
- moved U3 69.6 mm to (188.0, 76.2)
- moved C6 69.5 mm to (141.9, 78.2)
- moved J1 67.5 mm to (190.5, 83.8), turned to -90 degrees
- moved U2 67.0 mm to (194.3, 73.0), turned to -90 degrees
- moved C17 61.8 mm to (183.5, 74.9)
- moved R5 60.4 mm to (130.8, 79.5)
- moved C1 60.2 mm to (141.9, 76.2)
- moved R10 58.3 mm to (187.3, 72.4), turned to 180 degrees
- moved C9 56.5 mm to (183.5, 80.0), turned to 180 degrees
- moved C16 56.3 mm to (183.5, 77.5)
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Connections:
- C13 pad 1: -5V -> /Arduino Driver PCB/Vmeasure
- C14 pad 1: /Mid_Probe_2 -> GND
- C14 pad 2: Net-(U3B--) -> V_in
- C15 pad 1: +5V_Mid -> Net-(U3-SW)
- C15 pad 2: GND -> Net-(U3-BST)
- C16 pad 1: +5V_Mid -> GND
- C16 pad 2: GND -> +5V
- C17 pad 1: -5V -> GND
- C17 pad 2: GND -> +5V
- C19 pad 1: /Mid_TDS -> +3V3
- C20 pad 1: +5V -> /Bot_Temp
- C21 pad 1: /Arduino Driver PCB/Vmeasure -> +5V_Mid
- C22 pad 1: GND -> +5V_Mid
- C22 pad 2: V_in -> GND
- C23 pad 1: Net-(U5-SW) -> Net-(U5-C_{FLY+})
- C23 pad 2: Net-(U5-BST) -> Net-(U5-C_{FLY-})
- C24 pad 1: GND -> Net-(C24-Pad1)
- C24 pad 2: +5V -> /Mid_Probe_1
- C25 pad 1: GND -> -5V
- C25 pad 2: +5V -> GND
- C26 pad 1: +5V -> -5V
- C27 pad 1: +5V -> /Mid_Probe_2
- C27 pad 2: GND -> Net-(U7B--)
- C3 pad 1: +3V3 -> +5V
- C4 pad 1: +3V3 -> +5V
- C6 pad 1: +3V3 -> +5V_Bot
- C9 pad 1: +5V_Mid -> +5V
- D2 pad 1: Net-(D2-K) -> Net-(D13-A)
- D2 pad 2: Net-(D1-K) -> Net-(D2-A)
- D4 pad 1: V_in -> GND
- D4 pad 2: V_Supply -> Net-(D4-A)
- D5 pad 1: GND -> V_in
- D5 pad 2: Net-(D5-A) -> V_Supply
- J1 pad 1: GND -> /Arduino Driver PCB/UPDI
- J1 pad 2: /Bot_Temp -> +5V
- J2 pad 1: V_in -> GND
- J2 pad 2: GND -> /Bot_Temp
- J4 pad 1: unconnected-(J4-Pin_1-Pad1) -> V_in
- J4 pad 10: /Bot_SDA -> /SDA
- J4 pad 3: +5V_Bot -> V_Supply
- J4 pad 5: /Bot_Probe_1 -> +5V
- J4 pad 6: /Bot_Probe_2 -> /Top_TDS
- J4 pad 7: /Bot_Temp -> /Top_Temp
- J4 pad 8: /Bot_SCL -> /SCL
- J4 pad 9: /Bot_Status_LED -> /Top_TDS_OSC
- J5 pad 10: /Mid_SDA -> /Bot_SDA
- J5 pad 3: +5V_Mid -> +5V_Bot
- J5 pad 5: /Mid_Probe_1 -> /Bot_Probe_1
- J5 pad 6: /Mid_Probe_2 -> /Bot_Probe_2
- J5 pad 7: /Mid_Temp -> /Bot_Temp
- J5 pad 8: /Mid_SCL -> /Bot_SCL
- J5 pad 9: /Mid_Status_LED -> /Bot_Status_LED
- J7 pad 1: /Arduino Driver PCB/UPDI -> unconnected-(J7-Pin_1-Pad1)
- J7 pad 2: +5V -> GND
- J7 pad 3: /Arduino Driver PCB/Builtin_LED -> unconnected-(J7-Pin_3-Pad3)
- J7 pad 4: /Arduino Driver PCB/SERIAL_TX -> GND
- J7 pad 5: /Arduino Driver PCB/SERIAL_RX -> +5V_Mid
- J7 pad 6: GND -> /Mid_TDS
- R10 pad 1: Net-(U3B--) -> /Arduino Driver PCB/Vmeasure
- R10 pad 2: Net-(R10-Pad2) -> GND
- R11 pad 1: Net-(R10-Pad2) -> +5V
- R11 pad 2: Net-(U3C--) -> Net-(D10-A)
- R15 pad 1: Net-(U3D--) -> +5V_Mid
- R15 pad 2: Net-(R15-Pad2) -> /Function_Mid
- R16 pad 1: Net-(R15-Pad2) -> /Function_Mid
- R16 pad 2: /Mid_TDS -> GND
- R17 pad 1: V_in -> /Function_Mid
- R17 pad 2: /Arduino Driver PCB/Vmeasure -> GND
- R18 pad 1: /Arduino Driver PCB/Vmeasure -> +5V_Mid
- R18 pad 2: GND -> /Function_Mid
- R19 pad 1: /Arduino Driver PCB/Builtin_LED -> Net-(U7A--)
- R19 pad 2: Net-(D5-A) -> Net-(C24-Pad1)
- R20 pad 1: +5V -> /Mid_Probe_1
- R20 pad 2: Net-(D6-A) -> /Mid_Probe_2
- R5 pad 1: +3V3 -> /Bot_Temp
- R5 pad 2: /Pressure Transducer/AD/CS -> +5V_Bot
- R6 pad 1: unconnected-(R6-Pad1) -> /Mid_TDS_OSC
- R6 pad 2: Net-(U3A--) -> Net-(U7A--)
- R7 pad 1: Net-(U3A--) -> /Arduino Driver PCB/Builtin_LED
- R7 pad 2: Net-(C11-Pad1) -> Net-(D4-A)
- R9 pad 1: GND -> V_in
- R9 pad 2: Net-(U3B--) -> /Arduino Driver PCB/Vmeasure
- U2 pad 1: GND -> +5V
- U2 pad 2: -5V -> /Top_TDS
- U2 pad 3: Net-(U2-C_{FLY-}) -> /STATUS_LED
- U2 pad 4: +5V_Mid -> /Arduino Driver PCB/Builtin_LED
- U2 pad 5: +5V_Mid -> /Function
- U2 pad 6: Net-(U2-C_{FLY+}) -> /Arduino Driver PCB/SERIAL_RX
- U3 pad 1: Net-(C11-Pad1) -> +5V
- U3 pad 2: Net-(U3A--) -> V_in
- U3 pad 3: GND -> V_in
- U3 pad 4: +5V_Mid -> GND
- U3 pad 5: GND -> Net-(U3-SW)
- U3 pad 6: Net-(U3B--) -> Net-(U3-BST)
- U4 pad 1: +5V -> GND
- U4 pad 2: /Top_TDS -> +3V3
- U4 pad 3: /STATUS_LED -> +5V_Bot
- U5 pad 1: +5V -> GND
- U5 pad 2: V_in -> -5V
- U5 pad 3: V_in -> Net-(U5-C_{FLY-})
- U5 pad 4: GND -> +5V_Mid
- U5 pad 5: Net-(U5-SW) -> +5V_Mid
- U5 pad 6: Net-(U5-BST) -> Net-(U5-C_{FLY+})
Routing:
- net (no net): track 67.5 -> 0.00 mm, vias 2 -> 0
- net +5V_Mid: track 0.00 -> 36.3 mm, vias 0 -> 4
- net V_in: track 0.00 -> 31.5 mm, vias 0 -> 1
- net +5V: track 49.5 -> 79.1 mm, vias 6 -> 1
- net +3V3: track 38.1 -> 8.69 mm, vias 3 -> 0
- net +5V_Bot: track 0.00 -> 27.2 mm
- net /Arduino Driver PCB/SERIAL_RX: track 0.00 -> 27.0 mm
- net Net-(D2-K): track 26.9 -> 0.00 mm, vias 1 -> 0
- net /STATUS_LED: track 0.00 -> 23.1 mm
- net Net-(U7C--): track 0.00 -> 20.0 mm
- net /Arduino Driver PCB/SERIAL_TX: track 0.00 -> 19.1 mm, vias 0 -> 1
- net V_Supply: track 0.00 -> 18.6 mm, vias 0 -> 1
- net /Mid_TDS: track 0.00 -> 18.1 mm, vias 0 -> 1
- net /Arduino Driver PCB/UPDI: track 0.00 -> 18.0 mm, vias 0 -> 2
- net /Arduino Driver PCB/Builtin_LED: track 0.00 -> 15.9 mm, vias 0 -> 1
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- added copper zone on B.Cu, net V_Supply
- added copper zone on B.Cu, net V_in

Commit message: .
Parts:
- removed the REF** at (165.1, 71.1)
- added M1: MS5803-14BA, KiCad Footprints:MS5803-14BA, F.Cu at (139.7, 76.2)
- C33, C34, R21, R30, R31, R32, R33: moved to B.Cu
- moved R33 51.4 mm to (141.9, 70.0)
- moved R32 46.4 mm to (137.8, 70.0), turned to 180 degrees
- moved JP2 44.1 mm to (141.6, 71.1), turned to 180 degrees
- moved C34 42.6 mm to (137.8, 74.2), turned to 180 degrees
- moved C33 42.0 mm to (137.8, 72.1), turned to 180 degrees
- moved R31 42.0 mm to (137.8, 76.2)
- moved R30 40.2 mm to (137.8, 78.2)
- moved JP1 39.0 mm to (137.8, 71.1)
- moved R21 0.51 mm to (135.3, 83.9), turned to 90 degrees
Routing:
- net +3V3: track 8.69 -> 25.5 mm, vias 0 -> 1
- net /Bot_SDA: track 0.00 -> 13.0 mm, vias 0 -> 1
- net /Bot_SCL: track 0.00 -> 9.30 mm, vias 0 -> 1
- net /Pressure Transducer/AD/CS: track 0.00 -> 7.83 mm, vias 0 -> 1
- net /Pressure Transducer/PS: track 0.00 -> 7.76 mm, vias 0 -> 1
- net GND: track 40.6 -> 34.9 mm
- net Net-(D12-A): track 1.91 -> 3.84 mm, vias 0 -> 1
- net V_in: track 31.5 -> 33.1 mm
- net /Bot_Status_LED: track 3.15 -> 2.25 mm, vias 1 -> 0
